File: KiCad Getting Started.kicad_pcb (KiCad board)
At the start: 2 copper layers, 41.5 x 41 mm, 3 parts

Commit message: Done!
Parts:
- added SW1: M2011S3A1W03, getting-started:Switch_Toggle_SPST_NKK_M2011S3A1x03, F.Cu at (139.8, 116.5)
- moved R1 9.35 mm to (159.0, 107.2), turned to -90 degrees
Connections:
- D1 pad 2: VCC -> Net-(D1-A)
Routing:
- net Net-(D1-A): track 0.00 -> 15.1 mm
- net /led: track 18.1 -> 8.65 mm
- net VCC: track 16.5 -> 11.2 mm
- added copper zone on B.Cu, net GND
- added copper zone on F.Cu, net GND
- removed copper zone on B.Cu, net (none)
